File: pcb/pcb.kicad_pcb (KiCad board)
At the start: 2 copper layers, 190.5 x 85.7 mm, 98 parts, among them J1 OLED, SW1 RotaryEncoder_Switch, U1 Elite-C

Commit message: Routed LEDs.
Parts:
- moved D38 107.5 mm to (81.2, 75.6), turned to 0 degrees
- moved D41 107.4 mm to (186.8, 56.7)
- moved D39 48.4 mm to (138.7, 76.1), turned to 0 degrees
- moved D40 48.3 mm to (186.9, 78.8)
- moved C5 9.04 mm to (191.4, 56.7)
- moved C8 8.69 mm to (74.5, 77.3)
- moved C7 7.70 mm to (138.9, 80.0), turned to 0 degrees
Routing:
- net Net-(D36-Pad2): track 0.00 -> 81.8 mm, vias 0 -> 2
- net Net-(D39-Pad2): track 0.00 -> 62.0 mm, vias 0 -> 2
- net Net-(D39-Pad4): track 0.00 -> 53.9 mm
- net Net-(D38-Pad2): track 0.00 -> 49.0 mm
- net Net-(D35-Pad2): track 0.00 -> 48.6 mm
- net Net-(D34-Pad2): track 0.00 -> 46.8 mm
- net Net-(D42-Pad2): track 0.00 -> 35.7 mm, vias 0 -> 2
- net Net-(D41-Pad2): track 0.00 -> 30.9 mm
- net Net-(D41-Pad4): track 0.00 -> 25.6 mm
- net +5V: track 455.6 -> 444.4 mm, vias 2 -> 4
- net ROW3: track 193.0 -> 191.9 mm
- net GND: track 18.3 -> 17.2 mm
- net ROW2: track 243.6 -> 242.8 mm
- net COL2: track 170.6 -> 169.8 mm
